File: camera_capture_board/camera_capture_board.kicad_sch (KiCad schematic)
At the start: 2 parts, among them IC1 MIMXRT106FDVL6B

Commit message: Some updates
Parts:
- added C1: C, symbol Device:C
Connections:
- net VCC_SOC: now also IC1.H9 (VDD_SOC_IN_8), IC1.J5 (DCDC_SENSE), IC1.J9 (VDD_SOC_IN_9), C1.1
- net P0_MOSI: now reaches IC1.H10 (GPIO_AD_B0_01)
- net DCMI_D2: now reaches IC1.H11 (GPIO_AD_B1_13)
- net DCMI_D3: now reaches IC1.H12 (GPIO_AD_B1_12)
- net WIFI_CMD: now reaches IC1.H13 (GPIO_AD_B1_08)
- net BT_H_WAKE: now reaches IC1.H14 (GPIO_AD_B0_14)
- net at C34.2, IC1.H7 (VSS_9), IC1.H8 (VSS_10): now also C1.2; no longer IC1.H9 (VDD_SOC_IN_8)
- net SD_DAT0: now reaches IC1.J1 (GPIO_SD_B0_02)
- net DCMI_SCL: now reaches IC1.J11 (GPIO_AD_B1_00)
- net WIFI_D2: now reaches IC1.J12 (GPIO_AD_B1_06)
- net DCMI_D4: now reaches IC1.J13 (GPIO_AD_B1_11)
- net DCMI_D0: now reaches IC1.J14 (GPIO_AD_B1_15)
- net SD_DAT3: now reaches IC1.J2 (GPIO_SD_B0_05)
- net SD_CLK: now reaches IC1.J3 (GPIO_SD_B0_01)
- net SD_CMD: now reaches IC1.J4 (GPIO_SD_B0_00)
- net SD_DAT1: now reaches IC1.K1 (GPIO_SD_B0_03)
- net WIFI_D3: now reaches IC1.K10 (GPIO_AD_B1_07)
- net DCMI_SDA: now reaches IC1.K11 (GPIO_AD_B1_01)
- net BT_UART_RTS_N: now reaches IC1.K12 (GPIO_AD_B1_05)
- net P4_SCL: now reaches IC1.K14 (GPIO_AD_B0_12)
- net DCDC_PSWITCH: now reaches IC1.K3 (DCDC_PSWITCH)
- net PMIC_ON_REQ: now reaches IC1.K7 (PMIC_ON_REQ)
- net VDD_USB_CAP: now reaches IC1.K8 (VDD_USB_CAP)
- net DCMI_HSYNC: now reaches IC1.L10 (GPIO_AD_B0_15)
- net SD_CD: now reaches IC1.L11 (GPIO_AD_B1_02)
- net BT_UART_CTS_N: now reaches IC1.L12 (GPIO_AD_B1_04)
- net DCMI_D5: now reaches IC1.L13 (GPIO_AD_B1_10)
- net P5_SDA: now reaches IC1.L14 (GPIO_AD_B0_13)
- net P_FLASH_CE: now reaches IC1.L3 (GPIO_SD_B1_06)
- net P_FLASH_SCK: now reaches IC1.L4 (GPIO_SD_B1_07)
- net BT_D_WAKE: now reaches IC1.L5 (GPIO_SD_B1_00)
- net WAKEUP: now reaches IC1.L6 (WAKEUP)
- net PMIC_STBY_REQ: now reaches IC1.L7 (PMIC_STBY_REQ)
- net USB_D_P: now reaches IC1.L8 (USB_OTG1_DP)
- net DCDC_LP: now reaches IC1.M1 (DCDC_LP_1)
- net VDD_SNVS_CAP: now reaches IC1.M10 (VDD_SNVS_CAP)
- net P1_MISO: now reaches IC1.M11 (GPIO_AD_B0_02)
- net P6_ADC: now reaches IC1.M12 (GPIO_AD_B1_03)
- net WIFI_CLK: now reaches IC1.M13 (GPIO_AD_B1_09)
- net P2_SCLK: now reaches IC1.M14 (GPIO_AD_B0_00)
- net WIFI_D1: now reaches IC1.M3 (GPIO_SD_B1_02)
- net WIFI_D0: now reaches IC1.M4 (GPIO_SD_B1_03)
- net PWM_FSIN: now reaches IC1.M5 (GPIO_SD_B1_01)
- net ONOFF: now reaches IC1.M6 (ONOFF)
- net P12_RST_N: now reaches IC1.M7 (POR_B)
- net USB_D_N: now reaches IC1.M8 (USB_OTG1_DN)
- net P_FLASH_DQS: now reaches IC1.N3 (GPIO_SD_B1_05)
- net P_FLASH_IO1: now reaches IC1.N4 (GPIO_SD_B1_09)
