File: camera-control-board/camera-control-board.kicad_sch (KiCad schematic)
At the start: 16 parts, among them J1 DF12NB-36DS-0.5V_51_, U1 STM32H743IIT6, U2 IS42S32800J-7TLI, Y2 Crystal_GND2

Commit message: Changed IC, began USB.
I changed the correct IC, attempted to add USB. Want to make sure that we have the voltage protection circuit, not sure exactly how it works, will check soon.
Parts:
- removed U1: STM32H743IIT6, LQFP176-24x24mm, symbol 2024-09-28_20-43-17:STM32H743IIT6
- added C8: 2.2u, symbol Device:C
- added C9: 1u, symbol Device:C
- added CR1: USBLC6-2SC6, SOT23-6L_STM, symbol 2024-09-29_04-09-54:USBLC6-2SC6
- added J2: 10104110-0001LF, 10104110-0001LF:AMPHENOL_10104110-0001LF, symbol 10104110-0001LF:10104110-0001LF
- added R5, R6: 10K, symbol Device:R
- added U1: STM32H743IITx, Package_QFP:LQFP-176_24x24mm_P0.5mm, symbol MCU_ST_STM32H7:STM32H743IITx
- C7: value C -> 2.2u
Connections:
- net DAC: now also U1.51 (PA5)
- net DCMI_CLK: now also U1.119 (PA8)
- net DCMI_D0: now also U1.115 (PC6)
- net DCMI_D1: now also U1.116 (PC7)
- net DCMI_D2: now also U1.153 (PG10)
- net DCMI_D3: now also U1.154 (PG11)
- net DCMI_D4: now also U1.3 (PE4)
- net DCMI_D5: now also U1.164 (PB6)
- net DCMI_D6: now also U1.4 (PE5)
- net DCMI_D7: now also U1.5 (PE6)
- net DCMI_HSYNC: now also U1.50 (PA4)
- net DCMI_PCLK: now also U1.52 (PA6)
- net DCMI_PWDN: now also R6.1, U1.151 (PD7)
- net DCMI_RST: now also U1.121 (PA10)
- net DCMI_VSYNC: now also U1.165 (PB7)
- net DRAM_A0: now also U1.16 (PF0)
- net DRAM_A1: now also U1.17 (PF1)
- net DRAM_A10: now also U1.66 (PG0)
- net DRAM_A11: now also U1.67 (PG1)
- net DRAM_A2: now also U1.18 (PF2)
- net DRAM_A3: now also U1.19 (PF3)
- net DRAM_A4: now also U1.20 (PF4)
- net DRAM_A5: now also U1.21 (PF5)
- net DRAM_A6: now also U1.60 (PF12)
- net DRAM_A7: now also U1.63 (PF13)
- net DRAM_A8: now also U1.64 (PF14)
- net DRAM_A9: now also U1.65 (PF15)
- net DRAM_BA0: now also U1.108 (PG4)
- net DRAM_BA1: now also U1.109 (PG5)
- net DRAM_CAS: now also U1.160 (PG15)
- net DRAM_CLK: now also U1.112 (PG8)
- net DRAM_CLKE: now also U1.55 (PC5)
- net DRAM_CS: now also U1.54 (PC4)
- net DRAM_D0: now also U1.104 (PD14)
- net DRAM_D1: now also U1.105 (PD15)
- net DRAM_D10: now also U1.76 (PE13)
- net DRAM_D11: now also U1.77 (PE14)
- net DRAM_D12: now also U1.78 (PE15)
- net DRAM_D13: now also U1.96 (PD8)
- net DRAM_D14: now also U1.97 (PD9)
- net DRAM_D15: now also U1.98 (PD10)
- net DRAM_D16: now also U1.85 (PH8)
- net DRAM_D17: now also U1.86 (PH9)
- net DRAM_D18: now also U1.87 (PH10)
- net DRAM_D19: now also U1.88 (PH11)
- net DRAM_D2: now also U1.142 (PD0)
- net DRAM_D20: now also U1.89 (PH12)
- net DRAM_D21: now also U1.128 (PH13)
- net DRAM_D22: now also U1.129 (PH14)
- net DRAM_D23: now also U1.130 (PH15)
- net DRAM_D24: now also U1.131 (PI0)
- net DRAM_D25: now also U1.132 (PI1)
- net DRAM_D26: now also U1.133 (PI2)
- net DRAM_D27: now also U1.134 (PI3)
- net DRAM_D28: now also U1.175 (PI6)
- net DRAM_D29: now also U1.176 (PI7)
- net DRAM_D3: now also U1.143 (PD1)
- net DRAM_D30: now also U1.11 (PI9)
- net DRAM_D31: now also U1.12 (PI10)
- net DRAM_D4: now also U1.68 (PE7)
- net DRAM_D5: now also U1.69 (PE8)
- net DRAM_D6: now also U1.70 (PE9)
- net DRAM_D7: now also U1.73 (PE10)
- net DRAM_D8: now also U1.74 (PE11)
- net DRAM_D9: now also U1.75 (PE12)
- net DRAM_DQM0: now also U1.169 (PE0)
- net DRAM_DQM1: now also U1.170 (PE1)
- net DRAM_DQM2: now also U1.173 (PI4)
- net DRAM_DQM3: now also U1.174 (PI5)
- net DRAM_RAS: now also U1.59 (PF11)
- net DRAM_WE: now also U1.53 (PA7)
- net GND: now also C8.2, C9.2, CR1.2, J2.5 (GND), J2.SH1 (SHIELD), J2.SH2 (SHIELD__1), J2.SH3 (SHIELD__2), J2.SH4 (SHIELD__3), R5.1, U1.102 (VSS), U1.113 (VSS), U1.126 (VSS), U1.135 (VSS), U1.14 (VSS), U1.148 (VSS), U1.158 (VSS), U1.22 (VSS), U1.37 (VSSA), U1.48 (VSS), U1.61 (VSS), U1.71 (VSS), U1.90 (VSS); no longer C2.2, C3.1, Y2.2
- net I2C2_SCL: now also U1.79 (PB10)
- net I2C2_SDA: now also U1.80 (PB11)
- net LED_B: now also U1.34 (PC2_C)
- net LED_G: now also U1.33 (PC1)
- net LED_IR: now also U1.1 (PE2)
- net LED_R: now also U1.32 (PC0)
- net OSC_IN: now also U1.29 (PH0)
- net OSC_OUT: now also U1.30 (PH1)
- net SPI3_MISO: now also U1.162 (PB4)
- net SPI3_MOSI: now also U1.163 (PB5)
- net SPI3_SCLK/TRACESWO: now also U1.161 (PB3)
- net SPI3_SSEL: now also U1.138 (PA15)
- net VCC: now also J2.1 (VCC), R6.2, U1.103 (VDD), U1.114 (VDD33_USB), U1.127 (VDD), U1.136 (VDD), U1.149 (VDD), U1.15 (VDD), U1.159 (VDD), U1.171 (PDR_ON), U1.172 (VDD), U1.23 (VDD), U1.36 (VDD), U1.49 (VDD), U1.6 (VBAT), U1.62 (VDD), U1.72 (VDD), U1.82 (VDD), U1.91 (VDD)
- net VREF: now reaches C5.1, C6.1, L1.2
- net VREF: now also U1.38 (VREF+), U1.39 (VDDA)
- net at C7.1: now also U1.81 (VCAP)
- net NRST: no longer names the net of C4.1, R4.1
- net NRST: now also U1.31 (NRST)
- new net: C8.1, U1.125 (VCAP)
- new net: C2.2, C3.1, Y2.2
- new net: C9.1, CR1.5
- new net BOOT0: R5.2, U1.166 (BOOT0)
- new net FS_DM: CR1.6, U1.122 (PA11)
- new net FS_DM_C: CR1.1, J2.2 (D-)
- new net FS_DP: CR1.4, U1.123 (PA12)
- new net FS_DP_C: CR1.3, J2.3 (D+)
- new net I2C1_SCL: U1.167 (PB8)
- new net I2C1_SDA: U1.168 (PB9)
- new net P9: U1.107 (PG3)
- new net SDIO_CLK: U1.141 (PC12)
- new net SDIO_CMD: U1.144 (PD2)
- new net SDIO_D0: U1.117 (PC8)
- new net SDIO_D1: U1.118 (PC9)
- new net SDIO_D2: U1.139 (PC10)
- new net SDIO_D3: U1.140 (PC11)
- new net SD_CD: U1.111 (PG7)
- new net SPI2_MISO: U1.94 (PB14)
- new net SPI2_MOSI: U1.95 (PB15)
- new net SPI2_NSS: U1.92 (PB12)
- new net SPI2_SCLK: U1.93 (PB13)
- new net SWCLK: U1.137 (PA14)
- new net SWDIO: U1.124 (PA13)
- new net TIM4_CH1: U1.100 (PD12)
- new net TIM4_CH2: U1.101 (PD13)
- new net VBUS_R: U1.120 (PA9)
Other:
- note removed: "STM32-H7 MCU"
- moved on the sheet: C1, C2, C3, J1, R1, R2, R3, U2, Y2

Commit message: Removed USB Protection, added SD Card Circuit
Parts:
- removed CR1: USBLC6-2SC6, SOT23-6L_STM, symbol 2024-09-29_04-09-54:USBLC6-2SC6
- added J3: 104031-0811, 104031-0811:MOLEX_104031-0811, symbol 104031-0811:104031-0811
- added R7: R, symbol Device:R
- added RN1: EXB-V8V103JV, EXB38V472JV, symbol EXB-V8V103JV:EXB-V8V103JV
- C9: value 1u -> .1u
Connections:
- net FS_DM_C is gone; now on net FS_DM: J2.2 (D-)
- net FS_DP_C is gone; now on net FS_DP: J2.3 (D+)
- net GND: now also J3.10 (SW-2), J3.6 (VSS), J3.9 (SW-1), J3.G1 (GND), J3.G2 (GND__1), J3.G3 (GND__2), J3.G4 (GND__3)
- net SDIO_CLK: now also J3.5 (CLK)
- net SDIO_CMD: now also J3.3 (CMD), R7.2
- net VCC: now also C9.1, J3.4 (VDD), R7.1, RN1.1, RN1.2, RN1.3, RN1.4
- new net: J3.1 (DAT2), RN1.7
- new net: J3.2 (CD/DAT3), RN1.8
- new net: J3.7 (DAT0), RN1.5
- new net: J3.8 (DAT1), RN1.6
