File: camera-control-board.kicad_sch (KiCad schematic)
At the start: 58 parts, among them J1 DF12NB-36DS-0.5V_51_, J2 10104110-0001LF, J3 104031-0811, J4 02x05 M 1.27mm, J5 Conn_01x09, J6 USB_C_Receptacle_USB2.0, SW1 CAS-120TA, SW3 SW_Push, U1 STM32H743IITx, U2 IS42S32800J-7TLI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

Commit message: going to update pcb from schematic (will report back)
Parts:
- removed J2: 10104110-0001LF, Argus_Connectors:AMPHENOL_10104110-0001LF, symbol Argus_Connectors:10104110-0001LF
Connections:
- net VBUS: now also U4.1 (VIN), U4.3 (CE), VR1.1 (IN), VR1.3 (EN)
- net VCC: no longer U4.1 (VIN), U4.3 (CE), VR1.1 (IN), VR1.3 (EN)

Commit message: Layout finished; DRC checks next.
Connections:
- net VCC is gone; now on net +3.3V: R1.1, R6.2
Changed lines of the file:
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@@
 			)
 		)
-		(property "Value" "VCC"
+		(property "Value" "+3.3V"
 			(at 267.97 69.85 0)
 			(effects
@@
 		(on_board yes)
 		(dnp no)
-		(fields_autoplaced yes)
 		(property "Reference" "#PWR020"
 			(at 143.51 185.42 0)
@@
 			)
 		)
-		(property "Value" "VCC"
-			(at 143.51 176.53 0)
+		(property "Value" "+3.3V"
+			(at 140.462 177.292 0)
 			(effects
 				(font
 					(size 1.27 1.27)
 				)
+				(justify left)
 			)
 		)

Commit message: Minor Schematic cleanup
Parts:
- C18: footprint Capacitor_SMD:C_0201_0603Metric -> Capacitor_SMD:C_0805_2012Metric
- C2: footprint Capacitor_SMD:C_0603_1608Metric -> Capacitor_SMD:C_0805_2012Metric
- C5: value 1u -> 1uF
- C6: value .1u -> 0.1uF
- C7, C8: value 2.2u -> 2.2uF
- D2: value LED_RGBA -> 150141M173100; Field5 (none) -> LED_RGB
- J5: value Conn_01x09 -> 01x09 M 2.54mm
- J6: symbol Connector:USB_C_Receptacle_USB2.0 -> Connector:USB_C_Receptacle_USB2.0_16P
- R10: value 560 -> 560R
- R2, R3: value 4.7k -> 4.7K
- R7: value 10k -> 10K
Connections:
- no-connect marks 5 -> 42
Other:
- note removed: "Set for flight"
- moved on the sheet: C1, C10, C13, C14, C15, C16, C17, C19, C2, C3, C4, C5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

Commit message: added schematic for second set. Layout? Who's she..?
Parts:
- removed C11, C12: 4pF, Capacitor_SMD:C_0603_1608Metric, symbol Device:C_Small
- removed C13, C14, C15, C16, C17, C3: 0.1uF, Capacitor_SMD:C_0603_1608Metric, symbol Device:C_Small
- removed C18, C2: 47uF, Capacitor_SMD:C_0805_2012Metric, symbol Device:C_Polarized_Small_US
- removed C19: 1uF, Capacitor_SMD:C_0603_1608Metric, symbol Device:C_Small
- removed C5: 1uF, Capacitor_SMD:C_0603_1608Metric, symbol Device:C
- removed C6: 0.1uF, Capacitor_SMD:C_0603_1608Metric, symbol Device:C
- removed C7, C8: 2.2uF, Capacitor_SMD:C_0603_1608Metric, symbol Device:C
- removed D2: 150141M173100, LED_SMD:LED_RGB_Wuerth-PLCC4_3.2x2.8mm_150141M173100, symbol Device:LED_RGBA
- removed J1: DF12NB-36DS-0.5V_51_, Argus_Connectors:HRS_DF12NB-36DS-0.5V_51_, symbol Argus_Connectors:DF12NB-36DS-0.5V_51_
- removed J3: 104031-0811, Connector_Card:microSD_HC_Molex_104031-0811, symbol Argus_Connectors:USD-1040310811
- removed J4: 02x05 M 1.27mm, Connector_PinHeader_1.27mm:PinHeader_2x05_P1.27mm_Vertical_SMD, symbol Connector_Generic:Conn_02x05_Odd_Even
- removed J5: 01x09 M 2.54mm, Connector_PinHeader_2.54mm:PinHeader_1x09_P2.54mm_Vertical, symbol Connector_Generic:Conn_01x09
- removed L1: MPZ1608S181ATAH0, Argus_Misc:IND_1608_TDK, symbol Argus_Misc:MPZ1608S181ATAH0
- removed R1, R5, R6, R7: 10K, Resistor_SMD:R_0603_1608Metric, symbol Device:R
- removed R10: 560R, Resistor_SMD:R_0603_1608Metric, symbol Device:R
- removed R11: 1K, Resistor_SMD:R_0603_1608Metric, symbol Device:R_Small
- removed R16, R17, R18, R19, R20, R21: 10K, Resistor_SMD:R_0603_1608Metric, symbol Device:R_Small
- removed R2, R3: 4.7K, Resistor_SMD:R_0603_1608Metric, symbol Device:R
- removed RN2: 330R, Resistor_SMD:R_Array_Concave_4x0603, symbol Device:R_Pack04
- removed U1: STM32H743IITx, Package_QFP:LQFP-176_24x24mm_P0.5mm, symbol MCU_ST_STM32H7:STM32H743IITx
- removed U2: IS42S32800J-7TLI, Argus_ICs:SOP50P1176X120-86N, symbol Argus_ICs:IS42S32800J-7TLI
- removed U3: W25Q256JVEIQ TR, Argus_ICs:WSON8_E_WIN-L, symbol Argus_ICs:W25Q256JVEIQ_TR
- removed Y1: 12MHz/7pF, Crystal:Crystal_SMD_2520-4Pin_2.5x2.0mm, symbol Device:Crystal_GND24_Small
Connections:
- no-connect marks 42 -> 2
Other:
- added sheet uController_SD_RAM_Set_1 (uController_SD_RAM_Set_1.kicad_sch)
- added sheet uController_SD_RAM_Set_2 (uController_SD_RAM_Set_2.kicad_sch)
- note added: "USB-C Receptacle+Protection"
- note added: "uController-SD-RAM Sets"
- note removed: "32-Bit SDRAM"
- note removed: "Decoupling Caps"
- note removed: "Flash Memory"
- note removed: "Image Sensor Connector"
- note removed: "MCU (STM32H743IITx)"
- note removed: "SD Card Connector"
- note removed: "SWD Connector"
- note removed: "Status LEDs, IO Headers"
- note removed: "Status RGB LED"
- moved on the sheet: C1, C10, C4, C9, J6, R12, R13, R14, R15, R4, R8, R9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
